File: pcb_left/bluejay_left.kicad_sch (KiCad schematic)
At the start: 72 parts, among them J1 SJ-43514, SW1A KEYSW, SW1B KEYSW, SW1C KEYSW, SW1D KEYSW, SW1E KEYSW, SW2A KEYSW, SW2B KEYSW, SW2C KEYSW, SW2D KEYSW, SW2E KEYSW, SW2F KEYSW, SW3A KEYSW, SW3B KEYSW, SW3C KEYSW, SW3D KEYSW, SW3E KEYSW, SW3F KEYSW, SW4A KEYSW, SW4B KEYSW, SW4C KEYSW, SW4D KEYSW, SW4E KEYSW, SW4F KEYSW, SW5A KEYSW, SW5B KEYSW, SW5C KEYSW, SW5D KEYSW, U1 ATmega328P-PU, Y1 16MHz

Commit message: Further work on schematics
Parts:
- removed USB1: USB_B_Mini, symbol Connector:USB_B_Mini
- added USB1: USB_B_Mini, BlueJay footprints:USB_Mini_B_Female_548190519, symbol BlueJaySymbolLibrary:0548190519
- renumbered D1A to Da1, D2A to Da2, D3A to Da3, D4A to Da4, D5A to Da5, D1B to Db1, D2B to Db2, D3B to Db3, D4B to Db4, D5B to Db5, D1C to Dc1, D1D to Dd1, D1E to De1, SW1A to SWa1, SW2A to SWa2, SW3A to SWa3, SW4A to SWa4, SW5A to SWa5, SW1B to SWb1, SW2B to SWb2, SW3B to SWb3, SW4B to SWb4, SW5B to SWb5, SW1C to SWc1, SW1D to SWd1, SW1E to SWe1
Connections:
- net GND: now also USB1.1, USB1.SH
- net at DZ1.1 (K), R1.1, R2.2: now also USB1.4
- net at DZ2.1 (K), R3.2: now also USB1.3
- net at F1.2: now also USB1.5
Other:
- moved on the sheet: DZ1, DZ2, F1, J1, R1, R2, R3

Commit message: More work on schematics
Parts:
- C1, C2: footprint (none) -> BlueJay footprints:C_Disc_D3.0mm_W1.6mm_P2.50mm
- C3: footprint (none) -> BlueJay footprints:CP_Radial_D4.0mm_P1.50mm
- C4, C5: footprint (none) -> BlueJay footprints:C_Disc_D4.3mm_W1.9mm_P5.00mm
- F1: footprint (none) -> BlueJay footprints:polyfuse_5.1mm
- J1: footprint CUI_SJ-43514 -> BlueJay footprints:CUI_SJ-43514
- PB1, PB2: footprint (none) -> BlueJay footprints:SW_PUSH_6mm
- R1, R2, R3, R4: footprint (none) -> BlueJay footprints:R_Axial_DIN0204_L3.6mm_D1.6mm_P5.08mm_Horizontal
- SWa1, SWa2, SWa3, SWa4, SWa5, SWb1, SWb2, SWb3, SWb4, SWb5, SWc1, SWd1, SWe1: footprint (none) -> BlueJay footprints:Kailh_socket_MX
- SWc2: renamed from SW2C; footprint (none) -> BlueJay footprints:Kailh_socket_MX
- SWc3: renamed from SW3C; footprint (none) -> BlueJay footprints:Kailh_socket_MX
- SWc4: renamed from SW4C; footprint (none) -> BlueJay footprints:Kailh_socket_MX
- SWc5: renamed from SW5C; footprint (none) -> BlueJay footprints:Kailh_socket_MX
- SWd2: renamed from SW2D; footprint (none) -> BlueJay footprints:Kailh_socket_MX
- SWd3: renamed from SW3D; footprint (none) -> BlueJay footprints:Kailh_socket_MX
- SWd4: renamed from SW4D; footprint (none) -> BlueJay footprints:Kailh_socket_MX
- SWd5: renamed from SW5D; footprint (none) -> BlueJay footprints:Kailh_socket_MX
- SWe2: renamed from SW2E; footprint (none) -> BlueJay footprints:Kailh_socket_MX
- SWe3: renamed from SW3E; footprint (none) -> BlueJay footprints:Kailh_socket_MX
- SWe4: renamed from SW4E; footprint (none) -> BlueJay footprints:Kailh_socket_MX
- SWf2: renamed from SW2F; footprint (none) -> BlueJay footprints:Kailh_socket_MX
- SWf3: renamed from SW3F; footprint (none) -> BlueJay footprints:Kailh_socket_MX
- SWf4: renamed from SW4F; footprint (none) -> BlueJay footprints:Kailh_socket_MX
- USB1: footprint BlueJay footprints:USB_Mini_B_Female_548190519 -> digikey-footprints:USB_Mini_B_Female_548190519
- Y1: footprint (none) -> BlueJay footprints:Crystal_HC49-4H_Vertical
- renumbered D2C to Dc2, D3C to Dc3, D4C to Dc4, D5C to Dc5, D2D to Dd2, D3D to Dd3, D4D to Dd4, D5D to Dd5, D2E to De2, D3E to De3, D4E to De4, D2F to Df2, D3F to Df3, D4F to Df4

Commit message: Work on PCBs
Parts:
- USB1: footprint digikey-footprints:USB_Mini_B_Female_548190519 -> BlueJay footprints:USB_Mini_B_Female_548190519
Other:
- title: (none) -> BlueJay Left
Changed lines of the file:
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@@
 (kicad_sch (version 20211123) (generator eeschema)
   (paper "USLetter")
+  (title_block
+    (title "BlueJay Left")
+  )
   (junction (at 31.75 92.71) (diameter 0) (color 0 0 0 0)
   )
@@
       (effects (font (size 1.524 1.524)))
     )
-    (property "Footprint" "digikey-footprints:USB_Mini_B_Female_548190519" (id 2) (at 29.21 72.39 0)
+    (property "Footprint" "BlueJay footprints:USB_Mini_B_Female_548190519" (id 2) (at 29.21 72.39 0)
       (effects (font (size 1.524 1.524)) (justify left) hide)
     )
@@
     )
     (path "/65732213-2735-40de-8dfe-4a9a7e1cbc16"
-      (reference "USB1") (unit 1) (value "USB_B_Mini") (footprint "digikey-footprints:USB_Mini_B_Female_548190519")
+      (reference "USB1") (unit 1) (value "USB_B_Mini") (footprint "BlueJay footprints:USB_Mini_B_Female_548190519")
     )
     (path "/a4afee0d-8e42-4a5d-aac7-862e4657a136"
