File: pcb_left/bluejay_left.kicad_pcb (KiCad board)
At the start: 2 copper layers, 147 x 140.5 mm, 82 parts, among them J1 SJ-43514, U1 ATmega328P-PU, Y1 16MHz

Commit message: Produce test gerber files
Other:
- board text added: "BlueJay Keyboard"
- board text added: "https://github.com/JonathanFerron/BlueJay"
Changed lines of the file:
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@@
   (setup
     (stackup
-      (layer "F.SilkS" (type "Top Silk Screen"))
-      (layer "F.Mask" (type "Top Solder Mask") (thickness 0.01))
+      (layer "F.SilkS" (type "Top Silk Screen") (color "White"))
+      (layer "F.Mask" (type "Top Solder Mask") (color "Blue") (thickness 0.01))
       (layer "F.Cu" (type "copper") (thickness 0.035))
       (layer "dielectric 1" (type "core") (thickness 1.51) (material "FR4") (epsilon_r 4.5) (loss_tangent 0.02))
       (layer "B.Cu" (type "copper") (thickness 0.035))
-      (layer "B.Mask" (type "Bottom Solder Mask") (thickness 0.01))
-      (layer "B.SilkS" (type "Bottom Silk Screen"))
+      (layer "B.Mask" (type "Bottom Solder Mask") (color "Blue") (thickness 0.01))
+      (layer "B.SilkS" (type "Bottom Silk Screen") (color "White"))
       (copper_finish "None")
       (dielectric_constraints no)
     )
     (pad_to_mask_clearance 0)
-    (solder_mask_min_width 0.12)
     (pcbplotparams
-      (layerselection 0x00010fc_ffffffff)
+      (layerselection 0x00010f0_ffffffff)
       (disableapertmacros false)
       (usegerberextensions false)
@@
       (outputformat 1)
       (mirror false)
-      (drillshape 1)
+      (drillshape 0)
       (scaleselection 1)
-      (outputdirectory "")
+      (outputdirectory "../gerber/")
     )
   )
@@
     (property "Sheetname" "")
     (attr through_hole)
-    (fp_text reference "SWa5" (at 0 -8.255 -42) (layer "F.SilkS")
+    (fp_text reference "SWa5" (at 0 -8.255 -42 unlocked) (layer "F.SilkS")
       (effects (font (size 1 1) (thickness 0.15)))
     )
@@
     (property "exclude_from_bom" "")
     (attr exclude_from_pos_files exclude_from_bom)
-    (fp_text reference "H9" (at 0 -3.2) (layer "F.SilkS")
+    (fp_text reference "H9" (at 0 -3.2) (layer "F.SilkS") hide
       (effects (font (size 1 1) (thickness 0.15)))
     )
@@
       (effects (font (size 1 1) (thickness 0.15)))
     )
-    (fp_text value "100n" (at 2.54 0 90) (layer "F.SilkS")
+    (fp_text value "100n" (at 2.54 0 90) (layer "F.SilkS") hide
       (effects (font (size 0.8 1) (thickness 0.15)))
     )
@@
     (property "exclude_from_bom" "")
     (attr exclude_from_pos_files exclude_from_bom)
-    (fp_text reference "H8" (at 0 -3.2) (layer "F.SilkS")
+    (fp_text reference "H8" (at 0 -3.2) (layer "F.SilkS") hide
       (effects (font (size 1 1) (thickness 0.15)))
     )
@@
     (property "Sheetname" "")
     (attr through_hole)
-    (fp_text reference "SWd4" (at 0 -8.255) (layer "F.SilkS")
+    (fp_text reference "SWd4" (at -5.49 -7.91) (layer "F.SilkS")
       (effects (font (size 1 1) (thickness 0.15)))
     )
@@
     (property "exclude_from_bom" "")
     (attr exclude_from_pos_files exclude_from_bom)
-    (fp_text reference "H5" (at 0 -3.2) (layer "F.SilkS")
+    (fp_text reference "H5" (at 0 -3.2) (layer "F.SilkS") hide
       (effects (font (size 1 1) (thickness 0.15)))
     )
@@
     (property "exclude_from_bom" "")
     (attr exclude_from_pos_files exclude_from_bom)
-    (fp_text reference "H1" (at 0 -3.2) (layer "F.SilkS")
+    (fp_text reference "H1" (at 2.98 -2.4) (layer "F.SilkS") hide
       (effects (font (size 1 1) (thickness 0.15)))
     )
@@
     (property "exclude_from_bom" "")
     (attr exclude_from_pos_files exclude_from_bom)
-    (fp_text reference "H7" (at 0 -3.2) (layer "F.SilkS")
+    (fp_text reference "H7" (at 0 -3.2) (layer "F.SilkS") hide
       (effects (font (size 1 1) (thickness 0.15)))
     )
@@
     (property "Sheetname" "")
     (attr exclude_from_pos_files)
-    (fp_text reference "H2" (at 0 -3.2) (layer "F.SilkS")
+    (fp_text reference "H2" (at 0 -3.2) (layer "F.SilkS") hide
       (effects (font (size 1 1) (thickness 0.15)))
     )
@@
     (property "Sheetname" "")
     (attr exclude_from_pos_files)
-    (fp_text reference "H3" (at 0 -3.2) (layer "F.SilkS")
+    (fp_text reference "H3" (at 0 -3.2) (layer "F.SilkS") hide
       (effects (font (size 1 1) (thickness 0.15)))
     )
@@
     (property "Sheetname" "")
     (attr through_hole)
-    (fp_text reference "Dc4" (at 3.81 2.032) (layer "F.SilkS")
+    (fp_text reference "Dc4" (at 3.44 1.9) (layer "F.SilkS")
       (effects (font (size 0.8 0.8) (thickness 0.15)))
     )
@@
     (property "Sheetname" "")
     (attr through_hole)
-    (fp_text reference "R3" (at 2.54 -1.92) (layer "F.SilkS")
+    (fp_text reference "R3" (at 3.09 1.79) (layer "F.SilkS")
       (effects (font (size 1 1) (thickness 0.15)))
     )
-    (fp_text value "75R" (at 2.54 0) (layer "F.SilkS")
+    (fp_text value "75R" (at 2.54 0) (layer "F.SilkS") hide
       (effects (font (size 0.8 1) (thickness 0.15)))
     )
@@
       (effects (font (size 1 1) (thickness 0.15)))
     )
-    (fp_text value "100n" (at 2.54 0 90) (layer "F.SilkS")
+    (fp_text value "100n" (at 2.54 0 90) (layer "F.SilkS") hide
       (effects (font (size 0.8 1) (thickness 0.15)))
     )
@@
     (property "Sheetname" "")
     (attr through_hole)
-    (fp_text reference "SWb5" (at 0 -8.255 -28) (layer "F.SilkS")
+    (fp_text reference "SWb5" (at 0 -8.255 -28 unlocked) (layer "F.SilkS")
       (effects (font (size 1 1) (thickness 0.15)))
     )
@@
     (property "exclude_from_bom" "")
     (attr exclude_from_pos_files exclude_from_bom)
-    (fp_text reference "H6" (at 0 -3.2) (layer "F.SilkS")
+    (fp_text reference "H6" (at 0 -3.2) (layer "F.SilkS") hide
       (effects (font (size 1 1) (thickness 0.15)))
     )
@@
     (property "exclude_from_bom" "")
     (attr exclude_from_pos_files exclude_from_bom)
-    (fp_text reference "H4" (at 0 -3.2) (layer "F.SilkS")
+    (fp_text reference "H4" (at 0 -3.2) (layer "F.SilkS") hide
       (effects (font (size 1 1) (thickness 0.15)))
     )
@@
     (property "Sheetname" "")
     (attr through_hole)
-    (fp_text reference "SWc5" (at 0 -8.255 -14) (layer "F.SilkS")
+    (fp_text reference "SWc5" (at 0.026929 -8.484851 -14 unlocked) (layer "F.SilkS")
       (effects (font (size 1 1) (thickness 0.15)))
     )
@@
     (property "Sheetname" "")
     (attr through_hole)
-    (fp_text reference "R2" (at 2.54 2) (layer "F.SilkS")
+    (fp_text reference "R2" (at 2.45 -1.83) (layer "F.SilkS")
       (effects (font (size 1 1) (thickness 0.15)))
     )
-    (fp_text value "75R" (at 2.54 0) (layer "F.SilkS")
+    (fp_text value "75R" (at 2.54 0) (layer "F.SilkS") hide
       (effects (font (size 0.8 1) (thickness 0.15)))
     )
@@
   (gr_arc (start 49.7812 83.7263) (mid 48.888799 84.147698) (end 48.0112 83.6963) (layer "Edge.Cuts") (width 0.1))
   (gr_text "JLCJLCJLCJLC" (at -80.15 35.09) (layer "B.SilkS")
-    (effects (font (size 1 1) (thickness 0.2)) (justify mirror))
+    (effects (font (size 1 1) (thickness 0.15)) (justify mirror))
+  )
+  (gr_text "https://github.com/JonathanFerron/BlueJay" (at -51.27 32.63) (layer "B.SilkS")
+    (effects (font (size 1 1) (thickness 0.15)) (justify left mirror))
+  )
+  (gr_text "BlueJay Keyboard" (at -71.8 30.09) (layer "B.SilkS")
+    (effects (font (size 1 1) (thickness 0.15)) (justify left mirror))
   )
   (via (at 36 -40) (size 0.8) (drill 0.4) (layers "F.Cu" "B.Cu") (free) (net 1))

Commit message: Update schematics in preparation for review
Connections:
- net GND renamed Earth
Changed lines of the file:
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@@
   )
   (net 0 "")
-  (net 1 "GND")
+  (net 1 "Earth")
   (net 2 "Net-(C1-Pad1)")
   (net 3 "Net-(C2-Pad1)")
@@
       (net 3 "Net-(C2-Pad1)") (pintype "passive"))
     (pad "2" thru_hole circle (at 2.5 0) (size 1.6 1.6) (drill 0.8) (layers *.Cu *.Mask)
-      (net 1 "GND") (pintype "passive"))
+      (net 1 "Earth") (pintype "passive"))
     (model "${KICAD6_3DMODEL_DIR}/Capacitor_THT.3dshapes/C_Disc_D3.0mm_W1.6mm_P2.50mm.wrl"
       (offset (xyz 0 0 0))
@@
       (net 39 "/USBPRE_D+") (pinfunction "K") (pintype "passive"))
     (pad "2" thru_hole oval (at 6.35 0 90) (size 1.6 1.6) (drill 0.8) (layers *.Cu *.Mask)
-      (net 1 "GND") (pinfunction "A") (pintype "passive"))
+      (net 1 "Earth") (pinfunction "A") (pintype "passive"))
     (model "${KICAD6_3DMODEL_DIR}/Diode_THT.3dshapes/D_T-1_P5.08mm_Horizontal.step"
       (offset (xyz 1.3 0 0))
@@
       (net 4 "VCC") (pinfunction "VCC") (pintype "power_in"))
     (pad "8" thru_hole oval (at 0 17.78) (size 1.6 1.6) (drill 0.8) (layers *.Cu *.Mask)
-      (net 1 "GND") (pinfunction "GND") (pintype "power_in"))
+      (net 1 "Earth") (pinfunction "GND") (pintype "power_in"))
     (pad "9" thru_hole oval (at 0 20.32) (size 1.6 1.6) (drill 0.8) (layers *.Cu *.Mask)
       (net 2 "Net-(C1-Pad1)") (pinfunction "XTAL1/PB6") (pintype "bidirectional"))
@@
       (net 54 "unconnected-(U1-Pad21)") (pinfunction "AREF") (pintype "passive+no_connect"))
     (pad "22" thru_hole oval (at 7.62 15.24) (size 1.6 1.6) (drill 0.8) (layers *.Cu *.Mask)
-      (net 1 "GND") (pinfunction "GND") (pintype "passive"))
+      (net 1 "Earth") (pinfunction "GND") (pintype "passive"))
     (pad "23" thru_hole oval (at 7.62 12.7) (size 1.6 1.6) (drill 0.8) (layers *.Cu *.Mask)
       (net 34 "/colF") (pinfunction "PC0") (pintype "bidirectional"))
@@
       (net 4 "VCC") (pintype "passive"))
     (pad "2" thru_hole circle (at 5 0 90) (size 1.6 1.6) (drill 0.8) (layers *.Cu *.Mask)
-      (net 1 "GND") (pintype "passive"))
+      (net 1 "Earth") (pintype "passive"))
     (model "${KICAD6_3DMODEL_DIR}/Capacitor_THT.3dshapes/C_Disc_D4.3mm_W1.9mm_P5.00mm.wrl"
       (offset (xyz 0 0 0))
@@
       (net 38 "/USBPRE_D-") (pinfunction "K") (pintype "passive"))
     (pad "2" thru_hole oval (at 6.35 0 90) (size 1.6 1.6) (drill 0.8) (layers *.Cu *.Mask)
-      (net 1 "GND") (pinfunction "A") (pintype "passive"))
+      (net 1 "Earth") (pinfunction "A") (pintype "passive"))
     (model "${KICAD6_3DMODEL_DIR}/Diode_THT.3dshapes/D_T-1_P5.08mm_Horizontal.step"
       (offset (xyz 1.3 0 0))
@@
     (fp_circle (center 0 0) (end 2.45 0) (layer "F.CrtYd") (width 0.05) (fill none))
     (pad "1" thru_hole circle (at 0 0) (size 4.4 4.4) (drill 2.2) (layers *.Cu *.Mask)
-      (net 1 "GND") (pinfunction "1") (pintype "input"))
+      (net 1 "Earth") (pinfunction "1") (pintype "input"))
   )
   (footprint "BlueJay footprints:D_DO-35_SOD27_P5.08mm_Horizontal" (layer "F.Cu")
@@
     (fp_circle (center 0 0) (end 2.45 0) (layer "F.CrtYd") (width 0.05) (fill none))
     (pad "1" thru_hole circle (at 0 0) (size 4.4 4.4) (drill 2.2) (layers *.Cu *.Mask)
-      (net 1 "GND") (pinfunction "1") (pintype "input"))
+      (net 1 "Earth") (pinfunction "1") (pintype "input"))
   )
   (footprint "BlueJay footprints:D_DO-35_SOD27_P5.08mm_Horizontal" (layer "F.Cu")
@@
       (net 4 "VCC") (pintype "passive"))
     (pad "2" thru_hole circle (at 5 0 90) (size 1.6 1.6) (drill 0.8) (layers *.Cu *.Mask)
-      (net 1 "GND") (pintype "passive"))
+      (net 1 "Earth") (pintype "passive"))
     (model "${KICAD6_3DMODEL_DIR}/Capacitor_THT.3dshapes/C_Disc_D4.3mm_W1.9mm_P5.00mm.wrl"
       (offset (xyz 0 0 0))
@@
     (fp_line (start -8.8 3.85) (end 0.2 3.85) (layer "F.Fab") (width 0.1))
     (pad "1" thru_hole oval (at 0 -1.6 270) (size 1.65 1.1) (drill 0.7 (offset 0.275 0)) (layers *.Cu *.Mask)
-      (net 1 "GND") (pinfunction "GND") (pintype "passive"))
+      (net 1 "Earth") (pinfunction "GND") (pintype "passive"))
     (pad "2" thru_hole oval (at -1.2 -0.8 270) (size 1.65 1.1) (drill 0.7 (offset -0.275 0)) (layers *.Cu *.Mask)
       (net 57 "unconnected-(USB1-Pad2)") (pinfunction "ID") (pintype "passive+no_connect"))
@@
       (net 40 "Net-(F1-Pad2)") (pinfunction "VBUS") (pintype "passive"))
     (pad "SH" thru_hole oval (at -5.05 3.65 270) (size 2.7 1.7) (drill oval 1.9 0.7) (layers *.Cu *.Mask)
-      (net 1 "GND") (pinfunction "SHIELD") (pintype "passive"))
+      (net 1 "Earth") (pinfunction "SHIELD") (pintype "passive"))
     (pad "SH" thru_hole oval (at -5.05 -3.65 270) (size 2.7 1.7) (drill oval 1.9 0.7) (layers *.Cu *.Mask)
-      (net 1 "GND") (pinfunction "SHIELD") (pintype "passive"))
+      (net 1 "Earth") (pinfunction "SHIELD") (pintype "passive"))
     (model ":BlueJay3Dmodels:usb mini b connector 54819-0519.stp"
       (offset (xyz -9 0 2))
@@
       (net 2 "Net-(C1-Pad1)") (pintype "passive"))
     (pad "2" thru_hole circle (at 2.5 0) (size 1.6 1.6) (drill 0.8) (layers *.Cu *.Mask)
-      (net 1 "GND") (pintype "passive"))
+      (net 1 "Earth") (pintype "passive"))
     (model "${KICAD6_3DMODEL_DIR}/Capacitor_THT.3dshapes/C_Disc_D3.0mm_W1.6mm_P2.50mm.wrl"
       (offset (xyz 0 0 0))
@@
       (net 46 "/row1") (pinfunction "1") (pintype "passive"))
     (pad "2" thru_hole circle (at 0 4.5 180) (size 2 2) (drill 1.1) (layers *.Cu *.Mask)
-      (net 1 "GND") (pinfunction "2") (pintype "passive"))
+      (net 1 "Earth") (pinfunction "2") (pintype "passive"))
     (pad "2" thru_hole circle (at 6.5 4.5 180) (size 2 2) (drill 1.1) (layers *.Cu *.Mask)
-      (net 1 "GND") (pinfunction "2") (pintype "passive"))
+      (net 1 "Earth") (pinfunction "2") (pintype "passive"))
     (model "${KICAD6_3DMODEL_DIR}/Button_Switch_THT.3dshapes/SW_PUSH_6mm.wrl"
       (offset (xyz 0 0 0))
@@
       (net 43 "Net-(PB1-Pad1)") (pinfunction "1") (pintype "passive"))
     (pad "2" thru_hole circle locked (at 0 4.5 180) (size 2 2) (drill 1.1) (layers *.Cu *.Mask)
-      (net 1 "GND") (pinfunction "2") (pintype "passive"))
+      (net 1 "Earth") (pinfunction "2") (pintype "passive"))
     (pad "2" thru_hole circle locked (at 6.5 4.5 180) (size 2 2) (drill 1.1) (layers *.Cu *.Mask)
-      (net 1 "GND") (pinfunction "2") (pintype "passive"))
+      (net 1 "Earth") (pinfunction "2") (pintype "passive"))
     (model "${KISYS3DMOD}/Button_Switch_THT.3dshapes/SW_PUSH_6mm.wrl"
       (offset (xyz 0 0 0))
@@
     (pad "" np_thru_hole circle (at -2.6 0 270) (size 1.1 1.1) (drill 1.1) (layers *.Cu *.Mask))
     (pad "1" thru_hole rect (at -2.6 -4.8 270) (size 1.65 1.65) (drill 1.1) (layers *.Cu *.Mask)
-      (net 1 "GND") (pintype "passive"))
+      (net 1 "Earth") (pintype "passive"))
     (pad "2" thru_hole circle (at 2.4 3.6 270) (size 1.65 1.65) (drill 1.1) (layers *.Cu *.Mask)
       (net 4 "VCC") (pintype "passive"))
@@
       (net 4 "VCC") (pintype "passive"))
     (pad "2" thru_hole circle (at 1.5 0) (size 1.2 1.2) (drill 0.6) (layers *.Cu *.Mask)
-      (net 1 "GND") (pintype "passive"))
+      (net 1 "Earth") (pintype "passive"))
     (model "${KICAD6_3DMODEL_DIR}/Capacitor_THT.3dshapes/CP_Radial_D4.0mm_P1.50mm.wrl"
       (offset (xyz 0 0 0))
@@
   (segment (start 29.099627 53.794926) (end 13.060372 53.794926) (width 0.25) (layer "B.Cu") (net 50))
   (segment (start 8.548855 45.630026) (end 5.622629 42.7038) (width 0.25) (layer "B.Cu") (net 50))
-  (zone (net 1) (net_name "GND") (layers F&B.Cu) (hatch edge 0.508)
+  (zone (net 1) (net_name "Earth") (layers F&B.Cu) (hatch edge 0.508)
     (connect_pads (clearance 0.508))
     (min_thickness 0.254) (filled_areas_thickness no)
