File: pcb_right/bluejay_right.kicad_pcb (KiCad board)
At the start: 2 copper layers, 147 x 140.5 mm, 70 parts, among them J2 SJ-43514, U2 MCP23017

Commit message: Fine tune pcbs
Parts:
- moved De2 0.70 mm to (67.5, -45.0)
Routing:
- net GND: vias 0 -> 3
Changed lines of the file:
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@@
   )
   (footprint "BlueJay footprints:D_DO-35_SOD27_P5.08mm_Horizontal" (layer "F.Cu")
-    (at 66.8 -44.95 180)
+    (at 67.5 -44.95 180)
     (descr "Diode, DO-35_SOD27 series, Axial, Horizontal, pin pitch=7.62mm, , length*diameter=4*2mm^2, , http://www.diodes.com/_files/packages/DO-35.pdf")
     (tags "Diode DO-35_SOD27 series Axial Horizontal pin pitch 7.62mm  length 4mm diameter 2mm")
@@
   (gr_line (start -61.077843 -54.17) (end -61.077844 70.83) (layer "Edge.Cuts") (width 0.1))
   (gr_arc (start 83.927845 -56.17) (mid 85.346087 -55.593736) (end 85.927845 -54.17775) (layer "Edge.Cuts") (width 0.1))
-  (gr_text "JLCJLCJLCJLC" (at 79.63 35.43) (layer "B.Cu")
+  (gr_text "JLCJLCJLCJLC" (at 79.63 35.43) (layer "B.SilkS")
     (effects (font (size 1 1) (thickness 0.2)) (justify mirror))
   )
@@
   (segment (start -51.21 -4.505) (end -46.13 0.575) (width 0.4) (layer "B.Cu") (net 1))
   (segment (start -53.75 -4.505) (end -51.21 -4.505) (width 0.4) (layer "B.Cu") (net 1))
+  (via (at 77.75 -21.75) (size 0.8) (drill 0.4) (layers "F.Cu" "B.Cu") (free) (net 2))
+  (via (at -20.25 -51.25) (size 0.8) (drill 0.4) (layers "F.Cu" "B.Cu") (free) (net 2))
+  (via (at 64.75 -12.25) (size 0.8) (drill 0.4) (layers "F.Cu" "B.Cu") (free) (net 2))
   (segment (start -36.5675 19.5) (end -36.5675 4.5188) (width 0.25) (layer "F.Cu") (net 3))
   (segment (start -36.5863 -26.7437) (end -35.93 -27.4) (width 0.25) (layer "F.Cu") (net 3))
@@
   (segment (start -6.18 -52.45) (end -9.78 -52.45) (width 0.25) (layer "B.Cu") (net 15))
   (segment (start 1.47 -48.6) (end -2.33 -48.6) (width 0.25) (layer "B.Cu") (net 15))
-  (segment (start 19.4638 -52.45) (end 21.59 -50.3238) (width 0.25) (layer "B.Cu") (net 16))
-  (segment (start -1.1 -52.45) (end 19.4638 -52.45) (width 0.25) (layer "B.Cu") (net 16))
+  (segment (start 20.4138 -51.5) (end 21.59 -50.3238) (width 0.25) (layer "B.Cu") (net 16))
+  (segment (start -1.1 -52.45) (end -0.15 -51.5) (width 0.25) (layer "B.Cu") (net 16))
+  (segment (start -0.15 -51.5) (end 20.4138 -51.5) (width 0.25) (layer "B.Cu") (net 16))
   (segment (start 21.59 -31.2738) (end 21.59 -33.56) (width 0.25) (layer "F.Cu") (net 17))
   (segment (start 21.59 -33.56) (end 6.55 -48.6) (width 0.25) (layer "F.Cu") (net 17))
@@
   (segment (start -55.2 -23.735) (end -53.75 -22.285) (width 0.25) (layer "B.Cu") (net 21))
   (segment (start 40.83 -52.5) (end 39.58 -53.75) (width 0.25) (layer "B.Cu") (net 21))
-  (segment (start 41.954511 -51.375489) (end 40.83 -52.5) (width 0.25) (layer "B.Cu") (net 21))
-  (segment (start 51.455489 -51.375489) (end 41.954511 -51.375489) (width 0.25) (layer "B.Cu") (net 21))
-  (segment (start 52.58 -52.5) (end 51.455489 -51.375489) (width 0.25) (layer "B.Cu") (net 21))
+  (segment (start 51.33 -53.75) (end 42.08 -53.75) (width 0.25) (layer "B.Cu") (net 21))
+  (segment (start 52.58 -52.5) (end 51.33 -53.75) (width 0.25) (layer "B.Cu") (net 21))
+  (segment (start 42.08 -53.75) (end 40.83 -52.5) (width 0.25) (layer "B.Cu") (net 21))
   (segment (start 39.58 -53.75) (end -28.1 -53.75) (width 0.25) (layer "B.Cu") (net 21))
   (segment (start 40.64 -47.61) (end 35.75 -52.5) (width 0.25) (layer "F.Cu") (net 22))
@@
   (segment (start 12.065 40.1638) (end 12.065 33.3725) (width 0.25) (layer "F.Cu") (net 26))
   (segment (start 12.065 33.3725) (end 17.0375 28.4) (width 0.25) (layer "F.Cu") (net 26))
-  (segment (start 65.53 -44.95) (end 65 -45.48) (width 0.25) (layer "F.Cu") (net 27))
+  (segment (start 65.25 -51.5175) (end 64.3175 -52.45) (width 0.25) (layer "F.Cu") (net 27))
   (segment (start 73.78 -32) (end 73.15 -32.63) (width 0.25) (layer "F.Cu") (net 27))
+  (segment (start 66.23 -44.95) (end 65.25 -45.93) (width 0.25) (layer "F.Cu") (net 27))
   (segment (start 73.15 -32.63) (end 73.15 -39.88) (width 0.25) (layer "F.Cu") (net 27))
-  (segment (start 65 -45.48) (end 65 -51.7675) (width 0.25) (layer "F.Cu") (net 27))
-  (segment (start 65 -51.7675) (end 64.3175 -52.45) (width 0.25) (layer "F.Cu") (net 27))
+  (segment (start 65.25 -45.93) (end 65.25 -51.5175) (width 0.25) (layer "F.Cu") (net 27))
   (segment (start 73.15 -39.88) (end 72.58 -40.45) (width 0.25) (layer "F.Cu") (net 27))
   (segment (start 62.56798 -54.19952) (end -28.35048 -54.19952) (width 0.25) (layer "B.Cu") (net 27))
-  (segment (start 66.85 -44.95) (end 65.53 -44.95) (width 0.25) (layer "B.Cu") (net 27))
+  (segment (start 72.58 -40.45) (end 71.35 -40.45) (width 0.25) (layer "B.Cu") (net 27))
   (segment (start -55.70048 -21.69548) (end -53.75 -19.745) (width 0.25) (layer "B.Cu") (net 27))
+  (segment (start 66.85 -44.95) (end 66.23 -44.95) (width 0.25) (layer "B.Cu") (net 27))
   (segment (start -28.35048 -54.19952) (end -55.70048 -26.84952) (width 0.25) (layer "B.Cu") (net 27))
   (segment (start 64.3175 -52.45) (end 62.56798 -54.19952) (width 0.25) (layer "B.Cu") (net 27))
   (segment (start 71.35 -40.45) (end 66.85 -44.95) (width 0.25) (layer "B.Cu") (net 27))
-  (segment (start 72.58 -40.45) (end 71.35 -40.45) (width 0.25) (layer "B.Cu") (net 27))
   (segment (start -55.70048 -26.84952) (end -55.70048 -21.69548) (width 0.25) (layer "B.Cu") (net 27))
   (segment (start 58.9 -36.8263) (end 58.9 -52.1125) (width 0.25) (layer "F.Cu") (net 28))
   (segment (start 58.9 -52.1125) (end 59.2375 -52.45) (width 0.25) (layer "F.Cu") (net 28))
   (segment (start 59.69 -36.0363) (end 58.9 -36.8263) (width 0.25) (layer "F.Cu") (net 28))
+  (segment (start 61.75 -19.0463) (end 61.75 -44.35) (width 0.25) (layer "F.Cu") (net 29))
   (segment (start 59.69 -16.9863) (end 61.75 -19.0463) (width 0.25) (layer "F.Cu") (net 29))
-  (segment (start 61.75 -43.65) (end 60.45 -44.95) (width 0.25) (layer "F.Cu") (net 29))
-  (segment (start 61.75 -19.0463) (end 61.75 -43.65) (width 0.25) (layer "F.Cu") (net 29))
+  (segment (start 61.75 -44.35) (end 61.15 -44.95) (width 0.25) (layer "F.Cu") (net 29))
   (segment (start 59.69 -9.69) (end 67 -17) (width 0.25) (layer "F.Cu") (net 30))
   (segment (start 67 -39.95) (end 67.5 -40.45) (width 0.25) (layer "F.Cu") (net 30))
@@
   (segment (start 76.55 -26.65) (end 76.55 -36.25) (width 0.25) (layer "F.Cu") (net 34))
   (segment (start 80.45 0.3538) (end 80.45 -22.75) (width 0.25) (layer "F.Cu") (net 34))
-  (segment (start 81.9 -23.5875) (end 77.7375 -27.75) (width 0.25) (layer "F.Cu") (net 35))
-  (segment (start 78.74 21.1138) (end 81.9 17.9538) (width 0.25) (layer "F.Cu") (net 35))
-  (segment (start 81.9 17.9538) (end 81.9 -23.5875) (width 0.25) (layer "F.Cu") (net 35))
+  (segment (start 82.25 -23.2375) (end 77.7375 -27.75) (width 0.25) (layer "F.Cu") (net 35))
+  (segment (start 78.74 21.1138) (end 82.25 17.6038) (width 0.25) (layer "F.Cu") (net 35))
+  (segment (start 82.25 17.6038) (end 82.25 -23.2375) (width 0.25) (layer "F.Cu") (net 35))
   (segment (start -51.6 -34.31) (end -51.6 0.965) (width 0.25) (layer "F.Cu") (net 36))
   (segment (start -47.35 -45.2) (end -47.35 -43.44) (width 0.25) (layer "F.Cu") (net 36))
@@
     (connect_pads (clearance 0.508))
     (min_thickness 0.254) (filled_areas_thickness no)
-    (fill yes (thermal_gap 0.508) (thermal_bridge_width 0.508) (island_removal_mode 1) (island_area_min 0))
+    (fill yes (thermal_gap 0.508) (thermal_bridge_width 0.508))
     (polygon
       (pts

Commit message: Produce test gerber files
Other:
- board text added: "BlueJay Keyboard"
- board text added: "https://github.com/JonathanFerron/BlueJay"
Changed lines of the file:
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@@
   (setup
     (stackup
-      (layer "F.SilkS" (type "Top Silk Screen"))
-      (layer "F.Mask" (type "Top Solder Mask") (thickness 0.01))
+      (layer "F.SilkS" (type "Top Silk Screen") (color "White"))
+      (layer "F.Mask" (type "Top Solder Mask") (color "Blue") (thickness 0.01))
       (layer "F.Cu" (type "copper") (thickness 0.035))
       (layer "dielectric 1" (type "core") (thickness 1.51) (material "FR4") (epsilon_r 4.5) (loss_tangent 0.02))
       (layer "B.Cu" (type "copper") (thickness 0.035))
-      (layer "B.Mask" (type "Bottom Solder Mask") (thickness 0.01))
-      (layer "B.SilkS" (type "Bottom Silk Screen"))
+      (layer "B.Mask" (type "Bottom Solder Mask") (color "Blue") (thickness 0.01))
+      (layer "B.SilkS" (type "Bottom Silk Screen") (color "White"))
       (copper_finish "None")
       (dielectric_constraints no)
     )
     (pad_to_mask_clearance 0)
-    (solder_mask_min_width 0.12)
     (pcbplotparams
-      (layerselection 0x00010fc_ffffffff)
+      (layerselection 0x00010f0_ffffffff)
       (disableapertmacros false)
       (usegerberextensions false)
@@
       (outputformat 1)
       (mirror false)
-      (drillshape 1)
+      (drillshape 0)
       (scaleselection 1)
-      (outputdirectory "")
+      (outputdirectory "../gerber/")
     )
   )
@@
     (property "exclude_from_bom" "")
     (attr exclude_from_pos_files exclude_from_bom)
-    (fp_text reference "H5" (at 0 -3.2) (layer "F.SilkS")
+    (fp_text reference "H5" (at 0 -3.2) (layer "F.SilkS") hide
       (effects (font (size 1 1) (thickness 0.15)))
     )
@@
     (property "Sheetname" "")
     (attr exclude_from_pos_files)
-    (fp_text reference "H3" (at 0 -3.2) (layer "F.SilkS")
+    (fp_text reference "H3" (at 0 -3.2) (layer "F.SilkS") hide
       (effects (font (size 1 1) (thickness 0.15)))
     )
@@
     (property "exclude_from_bom" "")
     (attr exclude_from_pos_files exclude_from_bom)
-    (fp_text reference "H4" (at 0 -3.2) (layer "F.SilkS")
+    (fp_text reference "H4" (at 0 -3.2) (layer "F.SilkS") hide
       (effects (font (size 1 1) (thickness 0.15)))
     )
@@
     (property "Sheetname" "")
     (attr through_hole)
-    (fp_text reference "Dc4" (at 3.81 2.032) (layer "F.SilkS")
+    (fp_text reference "Dc4" (at 3.07 2.04) (layer "F.SilkS")
       (effects (font (size 0.8 0.8) (thickness 0.15)))
     )
@@
     (property "Sheetname" "")
     (attr exclude_from_pos_files)
-    (fp_text reference "H2" (at 0 -3.2) (layer "F.SilkS")
+    (fp_text reference "H2" (at 2.71 2.24) (layer "F.SilkS") hide
       (effects (font (size 1 1) (thickness 0.15)))
     )
@@
     (property "exclude_from_bom" "")
     (attr exclude_from_pos_files exclude_from_bom)
-    (fp_text reference "H1" (at 0 -3.2) (layer "F.SilkS")
+    (fp_text reference "H1" (at 0 -3.2) (layer "F.SilkS") hide
       (effects (font (size 1 1) (thickness 0.15)))
     )
@@
     (property "Sheetname" "")
     (attr through_hole)
-    (fp_text reference "SWd4" (at 0 -8.255) (layer "F.SilkS")
+    (fp_text reference "SWd4" (at 6.29 -8.2) (layer "F.SilkS")
       (effects (font (size 1 1) (thickness 0.15)))
     )
@@
     (property "exclude_from_bom" "")
     (attr exclude_from_pos_files exclude_from_bom)
-    (fp_text reference "H7" (at 0 -3.2) (layer "F.SilkS")
+    (fp_text reference "H7" (at 0 -3.2) (layer "F.SilkS") hide
       (effects (font (size 1 1) (thickness 0.15)))
     )
@@
     (property "exclude_from_bom" "")
     (attr exclude_from_pos_files exclude_from_bom)
-    (fp_text reference "H8" (at 0 -3.2) (layer "F.SilkS")
+    (fp_text reference "H8" (at 0 -3.2) (layer "F.SilkS") hide
       (effects (font (size 1 1) (thickness 0.15)))
     )
@@
     (property "Sheetname" "")
     (attr through_hole)
-    (fp_text reference "Dd4" (at 3.81 2.032) (layer "F.SilkS")
+    (fp_text reference "Dd4" (at 3.6675 -2.14) (layer "F.SilkS")
       (effects (font (size 0.8 0.8) (thickness 0.15)))
     )
@@
     (property "exclude_from_bom" "")
     (attr exclude_from_pos_files exclude_from_bom)
-    (fp_text reference "H9" (at 0 -3.2) (layer "F.SilkS")
+    (fp_text reference "H9" (at 0 -3.2) (layer "F.SilkS") hide
       (effects (font (size 1 1) (thickness 0.15)))
     )
@@
       (effects (font (size 1 1) (thickness 0.15)))
     )
-    (fp_text value "100n" (at 2.54 0 90) (layer "F.SilkS")
+    (fp_text value "100n" (at 2.54 0 90) (layer "F.SilkS") hide
       (effects (font (size 0.8 1) (thickness 0.15)))
     )
@@
     (property "Sheetname" "")
     (attr through_hole)
-    (fp_text reference "SWa5" (at 0 -8.255 42) (layer "F.SilkS")
+    (fp_text reference "SWa5" (at 2.868781 -8.491496 42) (layer "F.SilkS")
       (effects (font (size 1 1) (thickness 0.15)))
     )
@@
     (property "exclude_from_bom" "")
     (attr exclude_from_pos_files exclude_from_bom)
-    (fp_text reference "H6" (at 0 -3.2) (layer "F.SilkS")
+    (fp_text reference "H6" (at 0 -3.2) (layer "F.SilkS") hide
       (effects (font (size 1 1) (thickness 0.15)))
     )
@@
   (gr_line (start -61.077843 -54.17) (end -61.077844 70.83) (layer "Edge.Cuts") (width 0.1))
   (gr_arc (start 83.927845 -56.17) (mid 85.346087 -55.593736) (end 85.927845 -54.17775) (layer "Edge.Cuts") (width 0.1))
+  (gr_text "BlueJay Keyboard" (at 84.81 30.37) (layer "B.SilkS")
+    (effects (font (size 1 1) (thickness 0.15)) (justify left mirror))
+  )
   (gr_text "JLCJLCJLCJLC" (at 79.63 35.43) (layer "B.SilkS")
-    (effects (font (size 1 1) (thickness 0.2)) (justify mirror))
+    (effects (font (size 1 1) (thickness 0.15)) (justify mirror))
+  )
+  (gr_text "https://github.com/JonathanFerron/BlueJay" (at 84.81 32.78) (layer "B.SilkS")
+    (effects (font (size 1 1) (thickness 0.15)) (justify left mirror))
   )
   (segment (start -55.15 -39.25) (end -55.15 -40.65) (width 0.4) (layer "F.Cu") (net 1))

Commit message: Update schematics in preparation for review
Connections:
- net GND renamed Earth
Changed lines of the file:
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@@
   (net 0 "")
   (net 1 "VCC")
-  (net 2 "GND")
+  (net 2 "Earth")
   (net 3 "/colA")
   (net 4 "Net-(Da1-Pad2)")
@@
     (fp_circle (center 0 0) (end 2.45 0) (layer "F.CrtYd") (width 0.05) (fill none))
     (pad "1" thru_hole circle (at 0.4 -1) (size 4.4 4.4) (drill 2.2) (layers *.Cu *.Mask)
-      (net 2 "GND") (pinfunction "1") (pintype "input"))
+      (net 2 "Earth") (pinfunction "1") (pintype "input"))
   )
   (footprint "MountingHole:MountingHole_2.2mm_M2_Pad" (layer "F.Cu")
@@
     (pad "" np_thru_hole circle (at 2.4 0 270) (size 1.1 1.1) (drill 1.1) (layers *.Cu *.Mask))
     (pad "1" thru_hole rect (at -2.6 -4.8 270) (size 1.65 1.65) (drill 1.1) (layers *.Cu *.Mask)
-      (net 2 "GND") (pintype "passive"))
+      (net 2 "Earth") (pintype "passive"))
     (pad "2" thru_hole circle (at 2.4 3.6 270) (size 1.65 1.65) (drill 1.1) (layers *.Cu *.Mask)
       (net 1 "VCC") (pintype "passive"))
@@
       (net 1 "VCC") (pintype "passive"))
     (pad "2" thru_hole circle (at 1.5 0 180) (size 1.2 1.2) (drill 0.6) (layers *.Cu *.Mask)
-      (net 2 "GND") (pintype "passive"))
+      (net 2 "Earth") (pintype "passive"))
     (model "${KICAD6_3DMODEL_DIR}/Capacitor_THT.3dshapes/CP_Radial_D4.0mm_P1.50mm.wrl"
       (offset (xyz 0 0 0))
@@
     (fp_circle (center 0 0) (end 2.45 0) (layer "F.CrtYd") (width 0.05) (fill none))
     (pad "1" thru_hole circle (at 0 0) (size 4.4 4.4) (drill 2.2) (layers *.Cu *.Mask)
-      (net 2 "GND") (pinfunction "1") (pintype "input"))
+      (net 2 "Earth") (pinfunction "1") (pintype "input"))
   )
   (footprint "BlueJay footprints:D_DO-35_SOD27_P5.08mm_Horizontal" (layer "F.Cu")
@@
       (net 1 "VCC") (pintype "passive"))
     (pad "2" thru_hole circle (at 5 0 270) (size 1.6 1.6) (drill 0.8) (layers *.Cu *.Mask)
-      (net 2 "GND") (pintype "passive"))
+      (net 2 "Earth") (pintype "passive"))
     (model "${KICAD6_3DMODEL_DIR}/Capacitor_THT.3dshapes/C_Disc_D4.3mm_W1.9mm_P5.00mm.wrl"
       (offset (xyz 0 0 0))
@@
       (net 1 "VCC") (pinfunction "VDD") (pintype "power_in"))
     (pad "10" thru_hole oval (at 0 22.86) (size 1.6 1.6) (drill 0.8) (layers *.Cu *.Mask)
-      (net 2 "GND") (pinfunction "VSS") (pintype "power_in"))
+      (net 2 "Earth") (pinfunction "VSS") (pintype "power_in"))
     (pad "11" thru_hole oval (at 0 25.4) (size 1.6 1.6) (drill 0.8) (layers *.Cu *.Mask)
       (net 46 "unconnected-(U2-Pad11)") (pinfunction "NC") (pintype "no_connect"))
@@
       (net 47 "unconnected-(U2-Pad14)") (pinfunction "NC") (pintype "no_connect"))
     (pad "15" thru_hole oval (at 7.62 33.02) (size 1.6 1.6) (drill 0.8) (layers *.Cu *.Mask)
-      (net 2 "GND") (pinfunction "A0") (pintype "input"))
+      (net 2 "Earth") (pinfunction "A0") (pintype "input"))
     (pad "16" thru_hole oval (at 7.62 30.48) (size 1.6 1.6) (drill 0.8) (layers *.Cu *.Mask)
-      (net 2 "GND") (pinfunction "A1") (pintype "input"))
+      (net 2 "Earth") (pinfunction "A1") (pintype "input"))
     (pad "17" thru_hole oval (at 7.62 27.94) (size 1.6 1.6) (drill 0.8) (layers *.Cu *.Mask)
-      (net 2 "GND") (pinfunction "A2") (pintype "input"))
+      (net 2 "Earth") (pinfunction "A2") (pintype "input"))
     (pad "18" thru_hole oval (at 7.62 25.4) (size 1.6 1.6) (drill 0.8) (layers *.Cu *.Mask)
       (net 1 "VCC") (pinfunction "~{RESET}") (pintype "input"))
@@
   (segment (start -49.770753 68.691579) (end -52.800974 71.7218) (width 0.25) (layer "B.Cu") (net 42))
   (segment (start -32.955388 54.5) (end -35.827688 57.3723) (width 0.25) (layer "B.Cu") (net 42))
-  (zone (net 2) (net_name "GND") (layers F&B.Cu) (hatch edge 0.508)
+  (zone (net 2) (net_name "Earth") (layers F&B.Cu) (hatch edge 0.508)
     (connect_pads (clearance 0.508))
     (min_thickness 0.254) (filled_areas_thickness no)
