File: pcb_right/bluejay_right.kicad_pcb (KiCad board)
At the start: 2 copper layers, 148.7 x 142.4 mm, 67 parts, among them J2 SJ-43514, U2 MCP23017

Commit message: Update gerber files
Parts:
- removed G***: LOGO, BlueJay footprints:BlueJay_Logo_New_Small
- added Ref**: Val**, BlueJay footprints:BlueJay in Halfomania font, F.Cu at (-46.5, 36.0)
