File: pcb_left_test/bluejay_left.kicad_sch (KiCad schematic)
At the start: 81 parts, among them J1 SJ-43514, U1 ATmega328P-PU, Y1 16MHz

Commit message: Alternative approach to place diodes
Connections:
- net colA: now also U1.14 (PB0); no longer U1.15 (PB1)
- net colB: now also U1.13 (PD7); no longer U1.16 (PB2)
- net colC: now also U1.26 (PC3); no longer U1.14 (PB0)
- net colD: now also U1.25 (PC2); no longer PB2.1, U1.2 (PD0)
- net colE: now also U1.24 (PC1); no longer U1.25 (PC2)
- net colF: now also U1.23 (PC0); no longer U1.26 (PC3)
- net row1: now also PB2.1, U1.2 (PD0); no longer U1.3 (PD1)
- net row2: now also U1.3 (PD1); no longer U1.6 (PD4)
- net row3: now also U1.15 (PB1); no longer U1.11 (PD5)
- net row4: now also U1.16 (PB2); no longer U1.12 (PD6)
- net row5: now also U1.17 (PB3); no longer U1.13 (PD7)
