File: pcb_left_old/bluejay_left.kicad_sch (KiCad schematic)
At the start: 81 parts, among them J1 SJ-43514, U1 ATmega328P-PU, Y1 16MHz

Commit message: Create base pcb
Connections:
- net colA: now also U1.15 (PB1); no longer U1.14 (PB0)
- net colB: now also U1.16 (PB2); no longer U1.13 (PD7)
- net colC: now also U1.14 (PB0); no longer U1.26 (PC3)
- net colD: now also PB2.1, U1.2 (PD0); no longer U1.25 (PC2)
- net colE: now also U1.25 (PC2); no longer U1.24 (PC1)
- net colF: now also U1.26 (PC3); no longer U1.23 (PC0)
- net row1: now also U1.3 (PD1); no longer PB2.1, U1.2 (PD0)
- net row2: now also U1.6 (PD4); no longer U1.3 (PD1)
- net row3: now also U1.11 (PD5); no longer U1.15 (PB1)
- net row4: now also U1.12 (PD6); no longer U1.16 (PB2)
- net row5: now also U1.13 (PD7); no longer U1.17 (PB3)
- net USBPRE_D+: no longer names the net of DZ2.1 (K), R3.2, USB1.3 (D+)
- net USBPRE_D-: no longer names the net of DZ1.1 (K), R1.1, R2.2, USB1.4 (D-)
Changed lines of the file:
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@@
   )
   (no_connect (at 49.53 137.16))
+  (no_connect (at 49.53 132.08))
   (no_connect (at 49.53 134.62))
+  (no_connect (at 49.53 147.32))
+  (no_connect (at 49.53 149.86))
   (no_connect (at 19.05 124.46))
   (no_connect (at 31.75 74.93))
-  (no_connect (at 49.53 177.8))
-  (no_connect (at 49.53 180.34))
-  (no_connect (at 49.53 182.88))
   (wire (pts (xy 118.11 99.06) (xy 121.92 99.06))
     (stroke (width 0) (type default) (color 0 0 0 0))
@@
     (stroke (width 0) (type default) (color 0 0 0 0))
   )
+  (wire (pts (xy 49.53 182.88) (xy 53.34 182.88))
+    (stroke (width 0) (type default) (color 0 0 0 0))
+  )
   (wire (pts (xy 223.52 130.81) (xy 247.65 130.81))
     (stroke (width 0) (type default) (color 0 0 0 0))
@@
     (stroke (width 0) (type default) (color 0 0 0 0))
   )
-  (wire (pts (xy 49.53 147.32) (xy 53.34 147.32))
+  (wire (pts (xy 49.53 154.94) (xy 53.34 154.94))
     (stroke (width 0) (type default) (color 0 0 0 0))
   )
@@
     (stroke (width 0) (type default) (color 0 0 0 0))
   )
-  (wire (pts (xy 49.53 149.86) (xy 53.34 149.86))
+  (wire (pts (xy 49.53 152.4) (xy 53.34 152.4))
     (stroke (width 0) (type default) (color 0 0 0 0))
   )
@@
     (stroke (width 0) (type default) (color 0 0 0 0))
   )
+  (wire (pts (xy 49.53 177.8) (xy 53.34 177.8))
+    (stroke (width 0) (type default) (color 0 0 0 0))
+  )
   (wire (pts (xy 207.01 86.36) (xy 207.01 99.06))
     (stroke (width 0) (type default) (color 0 0 0 0))
@@
     (stroke (width 0) (type default) (color 0 0 0 0))
   )
-  (wire (pts (xy 49.53 132.08) (xy 53.34 132.08))
+  (wire (pts (xy 49.53 185.42) (xy 53.34 185.42))
     (stroke (width 0) (type default) (color 0 0 0 0))
   )
@@
     (stroke (width 0) (type default) (color 0 0 0 0))
   )
-  (wire (pts (xy 49.53 185.42) (xy 53.34 185.42))
-    (stroke (width 0) (type default) (color 0 0 0 0))
-  )
   (wire (pts (xy 182.88 128.27) (xy 212.09 128.27))
     (stroke (width 0) (type default) (color 0 0 0 0))
@@
     (stroke (width 0) (type default) (color 0 0 0 0))
   )
-  (wire (pts (xy 49.53 152.4) (xy 53.34 152.4))
-    (stroke (width 0) (type default) (color 0 0 0 0))
-  )
   (wire (pts (xy 93.98 182.88) (xy 93.98 184.15))
     (stroke (width 0) (type default) (color 0 0 0 0))
@@
     (stroke (width 0) (type default) (color 0 0 0 0))
   )
-  (wire (pts (xy 49.53 154.94) (xy 53.34 154.94))
-    (stroke (width 0) (type default) (color 0 0 0 0))
-  )
   (wire (pts (xy 55.88 137.16) (xy 57.15 137.16))
     (stroke (width 0) (type default) (color 0 0 0 0))
@@
     (stroke (width 0) (type default) (color 0 0 0 0))
   )
+  (wire (pts (xy 49.53 180.34) (xy 53.34 180.34))
+    (stroke (width 0) (type default) (color 0 0 0 0))
+  )
   (wire (pts (xy 97.79 88.9) (xy 121.92 88.9))
     (stroke (width 0) (type default) (color 0 0 0 0))
@@
     (effects (font (size 1.27 1.27)) (justify left bottom))
   )
-  (label "USBPRE_D-" (at 31.75 80.01 0)
-    (effects (font (size 1.27 1.27)) (justify left bottom))
-  )
   (label "USB_D+" (at 53.34 172.72 0)
     (effects (font (size 1.27 1.27)) (justify left bottom))
@@
     (effects (font (size 1.27 1.27)) (justify left bottom))
   )
-  (label "colF" (at 53.34 147.32 0)
+  (label "colF" (at 53.34 154.94 0)
     (effects (font (size 1.27 1.27)) (justify left bottom))
   )
@@
     (effects (font (size 1.27 1.27)) (justify left bottom))
   )
-  (label "row4" (at 53.34 129.54 0)
+  (label "row4" (at 53.34 182.88 0)
     (effects (font (size 1.27 1.27)) (justify left bottom))
   )
@@
     (effects (font (size 1.27 1.27)) (justify left bottom))
   )
-  (label "colC" (at 53.34 154.94 0)
-    (effects (font (size 1.27 1.27)) (justify left bottom))
-  )
-  (label "colE" (at 53.34 149.86 0)
-    (effects (font (size 1.27 1.27)) (justify left bottom))
-  )
-  (label "USBPRE_D+" (at 31.75 77.47 0)
-    (effects (font (size 1.27 1.27)) (justify left bottom))
-  )
-  (label "row3" (at 53.34 127 0)
+  (label "colC" (at 53.34 124.46 0)
+    (effects (font (size 1.27 1.27)) (justify left bottom))
+  )
+  (label "colE" (at 53.34 152.4 0)
+    (effects (font (size 1.27 1.27)) (justify left bottom))
+  )
+  (label "row3" (at 53.34 180.34 0)
     (effects (font (size 1.27 1.27)) (justify left bottom))
   )
@@
     (effects (font (size 1.27 1.27)) (justify left bottom))
   )
-  (label "row5" (at 53.34 132.08 0)
-    (effects (font (size 1.27 1.27)) (justify left bottom))
-  )
-  (label "colD" (at 53.34 152.4 0)
+  (label "row5" (at 53.34 185.42 0)
+    (effects (font (size 1.27 1.27)) (justify left bottom))
+  )
+  (label "colD" (at 53.34 167.64 0)
     (effects (font (size 1.27 1.27)) (justify left bottom))
   )
@@
     (effects (font (size 1.27 1.27)) (justify left bottom))
   )
-  (label "row2" (at 53.34 170.18 0)
+  (label "row2" (at 53.34 177.8 0)
     (effects (font (size 1.27 1.27)) (justify left bottom))
   )
@@
     (effects (font (size 1.27 1.27)) (justify left bottom))
   )
-  (label "row1" (at 53.34 167.64 0)
-    (effects (font (size 1.27 1.27)) (justify left bottom))
-  )
-  (label "colA" (at 53.34 124.46 0)
-    (effects (font (size 1.27 1.27)) (justify left bottom))
-  )
-  (label "colB" (at 53.34 185.42 0)
+  (label "row1" (at 53.34 170.18 0)
+    (effects (font (size 1.27 1.27)) (justify left bottom))
+  )
+  (label "colA" (at 53.34 127 0)
+    (effects (font (size 1.27 1.27)) (justify left bottom))
+  )
+  (label "colB" (at 53.34 129.54 0)
     (effects (font (size 1.27 1.27)) (justify left bottom))
   )
@@
   (symbol (lib_id "power:GND") (at 215.9 167.64 0) (unit 1)
     (in_bom yes) (on_board yes) (fields_autoplaced)
-    (property "Reference" "#PWR0115" (id 0) (at 215.9 173.99 0)
+    (property "Reference" "#PWR?" (id 0) (at 215.9 173.99 0)
       (effects (font (size 1.27 1.27)) hide)
     )
@@
     )
     (path "/aa799aa4-0b77-4e69-bd3a-b95b04823f1a"
-      (reference "#PWR0115") (unit 1) (value "GND") (footprint "")
+      (reference "#PWR?") (unit 1) (value "GND") (footprint "")
     )
     (path "/709a6874-5923-446e-9322-a60e23d13f71"
