File: pcb_plate/bluejay_plate.kicad_pcb (KiCad board)
At the start: 2 copper layers, 147.1 x 138.9 mm, 33 parts

Commit message: Fine tune pcbs
Connections:
- H4 pad 1: (no net) -> GND
Changed lines of the file:
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@@
   (footprint "BlueJay footprints:SW_Hole_TH" (layer "F.Cu")
     (at 19.05 2.3813)
-    (property "Sheetfile" "bluejay_left.kicad_sch")
+    (property "Sheetfile" "bluejay_plate.kicad_sch")
     (property "Sheetname" "")
     (attr through_hole)
@@
   (footprint "BlueJay footprints:SW_Hole_TH" (layer "F.Cu")
     (at 48.2012 71.0563 -42)
-    (property "Sheetfile" "bluejay_left.kicad_sch")
+    (property "Sheetfile" "bluejay_plate.kicad_sch")
     (property "Sheetname" "")
     (attr through_hole)
@@
   (footprint "BlueJay footprints:SW_Hole_TH" (layer "F.Cu")
     (at -76.2 -11.9063)
-    (property "Sheetfile" "bluejay_left.kicad_sch")
+    (property "Sheetfile" "bluejay_plate.kicad_sch")
     (property "Sheetname" "")
     (attr through_hole)
@@
   (footprint "BlueJay footprints:SW_Hole_TH" (layer "F.Cu")
     (at -19.05 -26.1938)
-    (property "Sheetfile" "bluejay_left.kicad_sch")
+    (property "Sheetfile" "bluejay_plate.kicad_sch")
     (property "Sheetname" "")
     (attr through_hole)
@@
   (footprint "BlueJay footprints:SW_Hole_TH" (layer "F.Cu")
     (at -38.1 -38.1)
-    (property "Sheetfile" "bluejay_left.kicad_sch")
+    (property "Sheetfile" "bluejay_plate.kicad_sch")
     (property "Sheetname" "")
     (attr through_hole)
@@
   (footprint "BlueJay footprints:SW_Hole_TH" (layer "F.Cu")
     (at -19.05 -7.1438)
-    (property "Sheetfile" "bluejay_left.kicad_sch")
+    (property "Sheetfile" "bluejay_plate.kicad_sch")
     (property "Sheetname" "")
     (attr through_hole)
@@
   (footprint "BlueJay footprints:SW_Hole_TH" (layer "F.Cu")
     (at -57.15 7.1438)
-    (property "Sheetfile" "bluejay_left.kicad_sch")
+    (property "Sheetfile" "bluejay_plate.kicad_sch")
     (property "Sheetname" "")
     (attr through_hole)
@@
   (footprint "BlueJay footprints:SW_Hole_TH" (layer "F.Cu")
     (at -19.05 11.9063)
-    (property "Sheetfile" "bluejay_left.kicad_sch")
+    (property "Sheetfile" "bluejay_plate.kicad_sch")
     (property "Sheetname" "")
     (attr through_hole)
@@
   (footprint "BlueJay footprints:SW_Hole_TH" (layer "F.Cu")
     (at -57.15 -11.9063)
-    (property "Sheetfile" "bluejay_left.kicad_sch")
+    (property "Sheetfile" "bluejay_plate.kicad_sch")
     (property "Sheetname" "")
     (attr through_hole)
@@
   (footprint "BlueJay footprints:SW_Hole_TH" (layer "F.Cu")
     (at -9.525 45.2438)
-    (property "Sheetfile" "bluejay_left.kicad_sch")
+    (property "Sheetfile" "bluejay_plate.kicad_sch")
     (property "Sheetname" "")
     (attr through_hole)
@@
   (footprint "BlueJay footprints:SW_Hole_TH" (layer "F.Cu")
     (at 19.05 21.4313)
-    (property "Sheetfile" "bluejay_left.kicad_sch")
+    (property "Sheetfile" "bluejay_plate.kicad_sch")
     (property "Sheetname" "")
     (attr through_hole)
@@
   (footprint "BlueJay footprints:SW_Hole_TH" (layer "F.Cu")
     (at 0 -38.1)
-    (property "Sheetfile" "bluejay_left.kicad_sch")
+    (property "Sheetfile" "bluejay_plate.kicad_sch")
     (property "Sheetname" "")
     (attr through_hole)
@@
   (footprint "BlueJay footprints:SW_Hole_TH" (layer "F.Cu")
     (at 0 -19.05)
-    (property "Sheetfile" "bluejay_left.kicad_sch")
+    (property "Sheetfile" "bluejay_plate.kicad_sch")
     (property "Sheetname" "")
     (attr through_hole)
@@
   (footprint "BlueJay footprints:SW_Hole_TH" (layer "F.Cu")
     (at 19.05 -16.6688)
-    (property "Sheetfile" "bluejay_left.kicad_sch")
+    (property "Sheetfile" "bluejay_plate.kicad_sch")
     (property "Sheetname" "")
     (attr through_hole)
@@
     (descr "Mounting Hole 2.2mm, M2")
     (tags "mounting hole 2.2mm m2")
-    (property "Sheetfile" "bluejay_left.kicad_sch")
+    (property "Sheetfile" "bluejay_plate.kicad_sch")
     (property "Sheetname" "")
     (property "exclude_from_bom" "")
@@
   (footprint "BlueJay footprints:SW_Hole_TH" (layer "F.Cu")
     (at -76.2 7.1438)
-    (property "Sheetfile" "bluejay_left.kicad_sch")
+    (property "Sheetfile" "bluejay_plate.kicad_sch")
     (property "Sheetname" "")
     (attr through_hole)
@@
   (footprint "BlueJay footprints:SW_Hole_TH" (layer "F.Cu")
     (at -38.1 19.05)
-    (property "Sheetfile" "bluejay_left.kicad_sch")
+    (property "Sheetfile" "bluejay_plate.kicad_sch")
     (property "Sheetname" "")
     (attr through_hole)
@@
     (descr "Mounting Hole 2.2mm, M2")
     (tags "mounting hole 2.2mm m2")
-    (property "Sheetfile" "bluejay_left.kicad_sch")
+    (property "Sheetfile" "bluejay_plate.kicad_sch")
     (property "Sheetname" "")
     (property "exclude_from_bom" "")
@@
   (footprint "BlueJay footprints:SW_Hole_TH" (layer "F.Cu")
     (at 0 19.05)
-    (property "Sheetfile" "bluejay_left.kicad_sch")
+    (property "Sheetfile" "bluejay_plate.kicad_sch")
     (property "Sheetname" "")
     (attr through_hole)
@@
   (footprint "BlueJay footprints:SW_Hole_TH" (layer "F.Cu")
     (at -57.15 26.1938)
-    (property "Sheetfile" "bluejay_left.kicad_sch")
+    (property "Sheetfile" "bluejay_plate.kicad_sch")
     (property "Sheetname" "")
     (attr through_hole)
@@
   (footprint "BlueJay footprints:SW_Hole_TH" (layer "F.Cu")
     (at 19.05 -35.7188)
-    (property "Sheetfile" "bluejay_left.kicad_sch")
+    (property "Sheetfile" "bluejay_plate.kicad_sch")
     (property "Sheetname" "")
     (attr through_hole)
@@
     (descr "Mounting Hole 2.2mm, M2")
     (tags "mounting hole 2.2mm m2")
-    (property "Sheetfile" "bluejay_left.kicad_sch")
+    (property "Sheetfile" "bluejay_plate.kicad_sch")
     (property "Sheetname" "")
     (property "exclude_from_bom" "")
@@
     (descr "Mounting Hole 2.2mm, M2")
     (tags "mounting hole 2.2mm m2")
-    (property "Sheetfile" "bluejay_left.kicad_sch")
+    (property "Sheetfile" "bluejay_plate.kicad_sch")
     (property "Sheetname" "")
     (attr exclude_from_pos_files)
@@
   (footprint "BlueJay footprints:SW_Hole_TH" (layer "F.Cu")
     (at 0 0)
-    (property "Sheetfile" "bluejay_left.kicad_sch")
+    (property "Sheetfile" "bluejay_plate.kicad_sch")
     (property "Sheetname" "")
     (attr through_hole)
@@
   (footprint "BlueJay footprints:SW_Hole_TH" (layer "F.Cu")
     (at 31.2712 57.8263 -28)
-    (property "Sheetfile" "bluejay_left.kicad_sch")
+    (property "Sheetfile" "bluejay_plate.kicad_sch")
     (property "Sheetname" "")
     (attr through_hole)
@@
     (descr "Mounting Hole 2.2mm, M2")
     (tags "mounting hole 2.2mm m2")
-    (property "Sheetfile" "bluejay_left.kicad_sch")
+    (property "Sheetfile" "bluejay_plate.kicad_sch")
     (property "Sheetname" "")
     (property "exclude_from_bom" "")
@@
     (descr "Mounting Hole 2.2mm, M2")
     (tags "mounting hole 2.2mm m2")
-    (property "Sheetfile" "bluejay_left.kicad_sch")
-    (property "Sheetname" "")
-    (property "exclude_from_bom" "")
-    (attr exclude_from_pos_files exclude_from_bom)
+    (property "Sheetfile" "bluejay_plate.kicad_sch")
+    (property "Sheetname" "")
+    (attr exclude_from_pos_files)
     (fp_text reference "H4" (at 0 -3.2) (layer "F.SilkS")
       (effects (font (size 1 1) (thickness 0.15)))
@@
     (fp_circle (center 0 0) (end 2.2 0) (layer "Cmts.User") (width 0.15) (fill none))
     (fp_circle (center 0 0) (end 2.45 0) (layer "F.CrtYd") (width 0.05) (fill none))
-    (pad "1" thru_hole circle (at 0 0) (size 4.4 4.4) (drill 2.2) (layers *.Cu *.Mask))
+    (pad "1" thru_hole circle (at 0 0) (size 4.4 4.4) (drill 2.2) (layers *.Cu *.Mask)
+      (net 1 "GND") (pinfunction "1") (pintype "input"))
   )
   (footprint "BlueJay footprints:SW_Hole_TH" (layer "F.Cu")
     (at -19.05 -45.2438)
-    (property "Sheetfile" "bluejay_left.kicad_sch")
+    (property "Sheetfile" "bluejay_plate.kicad_sch")
     (property "Sheetname" "")
     (attr through_hole)
@@
   (footprint "BlueJay footprints:SW_Hole_TH" (layer "F.Cu")
     (at -57.15 -30.9563)
-    (property "Sheetfile" "bluejay_left.kicad_sch")
+    (property "Sheetfile" "bluejay_plate.kicad_sch")
     (property "Sheetname" "")
     (attr through_hole)
@@
   (footprint "BlueJay footprints:SW_Hole_TH" (layer "F.Cu")
     (at -76.2 26.1938)
-    (property "Sheetfile" "bluejay_left.kicad_sch")
+    (property "Sheetfile" "bluejay_plate.kicad_sch")
     (property "Sheetname" "")
     (attr through_hole)
@@
   (footprint "BlueJay footprints:SW_Hole_TH" (layer "F.Cu")
     (at -38.1 0)
-    (property "Sheetfile" "bluejay_left.kicad_sch")
+    (property "Sheetfile" "bluejay_plate.kicad_sch")
     (property "Sheetname" "")
     (attr through_hole)
@@
   (footprint "BlueJay footprints:SW_Hole_TH" (layer "F.Cu")
     (at 11.6312 49.0163 -14)
-    (property "Sheetfile" "bluejay_left.kicad_sch")
+    (property "Sheetfile" "bluejay_plate.kicad_sch")
     (property "Sheetname" "")
     (attr through_hole)
@@
   (footprint "BlueJay footprints:SW_Hole_TH" (layer "F.Cu")
     (at -38.1 -19.05)
-    (property "Sheetfile" "bluejay_left.kicad_sch")
+    (property "Sheetfile" "bluejay_plate.kicad_sch")
     (property "Sheetname" "")
     (attr through_hole)
@@
   )
   (zone (net 1) (net_name "GND") (layers F&B.Cu) (hatch edge 0.508)
-    (connect_pads (clearance 0.508))
+    (connect_pads yes (clearance 0.508))
     (min_thickness 0.254) (filled_areas_thickness no)
     (fill yes (thermal_gap 0.508) (thermal_bridge_width 0.508))

Commit message: Produce test gerber files
Other:
- board text added: "BlueJay Keyboard"
Changed lines of the file:
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@@
     )
     (pad_to_mask_clearance 0)
-    (solder_mask_min_width 0.12)
     (pcbplotparams
-      (layerselection 0x00010fc_ffffffff)
+      (layerselection 0x00010f0_ffffffff)
       (disableapertmacros false)
       (usegerberextensions false)
@@
       (outputformat 1)
       (mirror false)
-      (drillshape 1)
+      (drillshape 0)
       (scaleselection 1)
-      (outputdirectory "")
+      (outputdirectory "../gerber/")
     )
   )
@@
     (property "exclude_from_bom" "")
     (attr exclude_from_pos_files exclude_from_bom)
-    (fp_text reference "H8" (at 0 -3.2) (layer "F.SilkS")
+    (fp_text reference "H8" (at 0 -3.2) (layer "F.SilkS") hide
       (effects (font (size 1 1) (thickness 0.15)))
     )
@@
     (property "exclude_from_bom" "")
     (attr exclude_from_pos_files exclude_from_bom)
-    (fp_text reference "H5" (at 0 -3.2) (layer "F.SilkS")
+    (fp_text reference "H5" (at 0 -3.2) (layer "F.SilkS") hide
       (effects (font (size 1 1) (thickness 0.15)))
     )
@@
     (property "exclude_from_bom" "")
     (attr exclude_from_pos_files exclude_from_bom)
-    (fp_text reference "H7" (at 0 -3.2) (layer "F.SilkS")
+    (fp_text reference "H7" (at 0 -3.2) (layer "F.SilkS") hide
       (effects (font (size 1 1) (thickness 0.15)))
     )
@@
     (property "Sheetname" "")
     (attr exclude_from_pos_files)
-    (fp_text reference "H3" (at 0 -3.2) (layer "F.SilkS")
+    (fp_text reference "H3" (at 0 -3.2) (layer "F.SilkS") hide
       (effects (font (size 1 1) (thickness 0.15)))
     )
@@
     (property "exclude_from_bom" "")
     (attr exclude_from_pos_files exclude_from_bom)
-    (fp_text reference "H6" (at 0 -3.2) (layer "F.SilkS")
+    (fp_text reference "H6" (at 0 -3.2) (layer "F.SilkS") hide
       (effects (font (size 1 1) (thickness 0.15)))
     )
@@
     (property "Sheetname" "")
     (attr exclude_from_pos_files)
-    (fp_text reference "H4" (at 0 -3.2) (layer "F.SilkS")
+    (fp_text reference "H4" (at 0 -3.2) (layer "F.SilkS") hide
       (effects (font (size 1 1) (thickness 0.15)))
     )
@@
   (gr_arc (start 8.43845 -47.625422) (mid 9.218647 -47.301388) (end 9.52845 -46.515422) (layer "Edge.Cuts") (width 0.1))
   (gr_text "JLCJLCJLCJLC" (at -19 -35.74) (layer "F.SilkS")
-    (effects (font (size 1 1) (thickness 0.2)))
+    (effects (font (size 1 1) (thickness 0.15)))
+  )
+  (gr_text "BlueJay Keyboard" (at -19.32 32.25) (layer "F.SilkS")
+    (effects (font (size 1.5 1.5) (thickness 0.25)))
   )
   (zone (net 1) (net_name "GND") (layers F&B.Cu) (hatch edge 0.508)

Commit message: Update schematics in preparation for review
Connections:
- net GND renamed Earth
Changed lines of the file:
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@@
   )
   (net 0 "")
-  (net 1 "GND")
+  (net 1 "Earth")
   (footprint "BlueJay footprints:SW_Hole_TH" (layer "F.Cu")
     (at 19.05 2.3813)
@@
     (fp_circle (center 0 0) (end 2.45 0) (layer "F.CrtYd") (width 0.05) (fill none))
     (pad "1" thru_hole circle (at 0 0) (size 4.4 4.4) (drill 2.2) (layers *.Cu *.Mask)
-      (net 1 "GND") (pinfunction "1") (pintype "input"))
+      (net 1 "Earth") (pinfunction "1") (pintype "input"))
   )
   (footprint "BlueJay footprints:SW_Hole_TH" (layer "F.Cu")
@@
     (fp_circle (center 0 0) (end 2.45 0) (layer "F.CrtYd") (width 0.05) (fill none))
     (pad "1" thru_hole circle (at 0 0) (size 4.4 4.4) (drill 2.2) (layers *.Cu *.Mask)
-      (net 1 "GND") (pinfunction "1") (pintype "input"))
+      (net 1 "Earth") (pinfunction "1") (pintype "input"))
   )
   (footprint "BlueJay footprints:SW_Hole_TH" (layer "F.Cu")
@@
     (effects (font (size 1.5 1.5) (thickness 0.25)))
   )
-  (zone (net 1) (net_name "GND") (layers F&B.Cu) (hatch edge 0.508)
+  (zone (net 1) (net_name "Earth") (layers F&B.Cu) (hatch edge 0.508)
     (connect_pads yes (clearance 0.508))
     (min_thickness 0.254) (filled_areas_thickness no)

Commit message: Fine tuning of schematics and pcbs in prep for review
Connections:
- net Earth renamed GND
Changed lines of the file:
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@@
   )
   (net 0 "")
-  (net 1 "Earth")
+  (net 1 "GND")
   (footprint "BlueJay footprints:SW_Hole_TH" (layer "F.Cu")
     (at 19.05 2.3813)
@@
     (fp_circle (center 0 0) (end 2.45 0) (layer "F.CrtYd") (width 0.05) (fill none))
     (pad "1" thru_hole circle (at 0 0) (size 4.4 4.4) (drill 2.2) (layers *.Cu *.Mask)
-      (net 1 "Earth") (pinfunction "1") (pintype "input"))
+      (net 1 "GND") (pinfunction "1") (pintype "input"))
   )
   (footprint "BlueJay footprints:SW_Hole_TH" (layer "F.Cu")
@@
     (fp_circle (center 0 0) (end 2.45 0) (layer "F.CrtYd") (width 0.05) (fill none))
     (pad "1" thru_hole circle (at 0 0) (size 4.4 4.4) (drill 2.2) (layers *.Cu *.Mask)
-      (net 1 "Earth") (pinfunction "1") (pintype "input"))
+      (net 1 "GND") (pinfunction "1") (pintype "input"))
   )
   (footprint "BlueJay footprints:SW_Hole_TH" (layer "F.Cu")
@@
     (effects (font (size 1.5 1.5) (thickness 0.25)))
   )
-  (zone (net 1) (net_name "Earth") (layers F&B.Cu) (hatch edge 0.508)
+  (zone (net 1) (net_name "GND") (layers F&B.Cu) (hatch edge 0.508)
     (connect_pads yes (clearance 0.508))
     (min_thickness 0.254) (filled_areas_thickness no)
